File: KAKATA_MOD_FUNCIONES_PCB/KAKATA_MOD_FUNCIONES.kicad_sch (KiCad schematic)
At the start: 61 parts, among them J1 DB128L-5.08-2P-BK-S, J2 Screw_Terminal_01x02, J3 Screw_Terminal_01x02, J4 Screw_Terminal_01x02, J5 DB125-2.54-10P-GN, J6 DB125-2.54-4P-GN, Q1 MMUN2215L, Q2 MMUN2215L, Q3 MMUN2215L, U1 ESP32-S3-WROOM-1(N16R8), U2 PS-TO220, U3 PS-TO220, U4 TYPE-C 16PLT-H10.0

Commit message: Btn's BOOT y RST agregados. Encendido secuencial implementado
Parts:
- removed C1: 1uF, Capacitor_SMD_AKL:C_0603_1608Metric, symbol PCM_Capacitor_US_AKL:C_0603
- removed D2: B0540LW, Diode_SMD_AKL:D_SOD-123, symbol PCM_Diode_Schottky_AKL:B0540LW
- removed D4: B0540LW, PCM_Diode_SMD_AKL:D_SOD-123, symbol PCM_Diode_Schottky_AKL:B0540LW
- removed J2, J3, J4: Screw_Terminal_01x02, EasyEDA:CONN-TH_2P-P5.08_DIBO_DB128V-5.08, symbol Connector:Screw_Terminal_01x02
- removed J6: DB125-2.54-4P-GN, EasyEDA:CONN-TH_DB125-2.54-4P-GN, symbol EasyEDA:DB125-2.54-4P-GN
- removed Q1, Q2, Q3: MMUN2215L, PCM_Package_TO_SOT_SMD_AKL:SOT-23, symbol PCM_Transistor_BJT_Pre-Biased_AKL:MMUN2215L
- removed TP1: TestPoint_Hole1, 4ms_TestPoint:TestPoint_WireHole, symbol MG_ELECTROMECANICAL:TestPoint_Hole1
- removed U4: TYPE-C 16PLT-H10.0, EasyEDA:TYPE-C-SMD_USB4120-03-C, symbol EasyEDA:TYPE-C16PLT-H10.0
- added C2: 0.1uF, EasyEDA:C0603, symbol PCM_Capacitor_US_AKL:C_0603
- added C3: 1uF, EasyEDA:C0603, symbol PCM_Capacitor_US_AKL:C_0603
- added D2: SS24-SMB, EasyEDA:SMB_L4.3-W3.6-LS5.3-RD, symbol EasyEDA:SS24-SMB
- added D3: B0540W, EasyEDA:SOD-123_L2.7-W1.6-LS3.7-FD, symbol EasyEDA:B0540W_C7420325
- added J2, J3, J4: Conn_01x02_Socket, Connector_Molex:Molex_KK-254_AE-6410-02A_1x02_P2.54mm_Vertical, symbol Connector:Conn_01x02_Socket
- added J5: Conn_01x03_Socket, Connector_Molex:Molex_KK-254_AE-6410-03A_1x03_P2.54mm_Vertical, symbol Connector:Conn_01x03_Socket
- added Q2: AOD4185_C400894, EasyEDA:TO-252-3_L6.6-W6.1-P4.57-LS9.9-BR-CW, symbol EasyEDA:AOD4185_C400894
- added Q3, Q4, Q5: MMUN2215LT1G, EasyEDA:SOT-23-3_L2.9-W1.3-P1.90-LS2.4-BR, symbol EasyEDA:MMUN2215LT1G
- added R3: 10k, EasyEDA:R0603, symbol PCM_Resistor_US_AKL:R_0603
- added SW1, SW2: TS-1088-AR02016, EasyEDA:SW-SMD_L3.9-W3.0-P4.45, symbol EasyEDA:TS-1088-AR02016
- added TP1, TP2, TP3: TestPoint, TestPoint:TestPoint_Pad_D2.0mm, symbol Connector:TestPoint
- added USB1: TYPE-C 16PIN 2MD, EasyEDA:USB-C-SMD_TYPE-C-6PIN-2MD-073, symbol EasyEDA:TYPE-C16PIN2MD
- C1: renamed from C2; footprint Capacitor_SMD_AKL:CP_Elec_6.3x7.7 -> EasyEDA:CAP-SMD_BD6.3-L6.6-W6.6-LS7.2-FD; symbol Capacitor_AKL:CP_SMD_D6.3mm_H7.7mm -> PCM_Capacitor_US_AKL:CP_SMD_D6.3mm_H7.7mm
- C10: renamed from C9; footprint PCM_Capacitor_SMD_AKL:C_0805_2012Metric -> EasyEDA:C0805
- C11: renamed from C10; footprint PCM_Capacitor_SMD_AKL:C_0603_1608Metric -> EasyEDA:C0603
- C12: renamed from C11; footprint PCM_Capacitor_SMD_AKL:C_0603_1608Metric -> EasyEDA:C0603
- C13: renamed from C12; footprint PCM_Capacitor_SMD_AKL:C_0603_1608Metric -> EasyEDA:C0603
- C14: renamed from C13; footprint PCM_Capacitor_SMD_AKL:C_0603_1608Metric -> EasyEDA:C0603
- C15: renamed from C14; footprint PCM_Capacitor_SMD_AKL:C_0603_1608Metric -> EasyEDA:C0603
- C16: renamed from C15; footprint PCM_Capacitor_SMD_AKL:C_0603_1608Metric -> EasyEDA:C0603
- C4: renamed from C3; footprint PCM_Capacitor_SMD_AKL:C_0603_1608Metric -> EasyEDA:C0603
- C5: renamed from C4; footprint PCM_Capacitor_SMD_AKL:C_0603_1608Metric -> EasyEDA:C0603
- C6: renamed from C5; footprint PCM_Capacitor_SMD_AKL:C_0603_1608Metric -> EasyEDA:C0603
- C7: renamed from C6; footprint PCM_Capacitor_SMD_AKL:C_0603_1608Metric -> EasyEDA:C0603
- C8: renamed from C7; footprint PCM_Capacitor_SMD_AKL:C_0603_1608Metric -> EasyEDA:C0603
- C9: renamed from C8; footprint PCM_Capacitor_SMD_AKL:C_0603_1608Metric -> EasyEDA:C0603
- D1: footprint Diode_SMD_AKL:D_SOD-323_TVS -> Diode_SMD:D_SOD-323; LCSC Part C22466620 -> (none)
- D4: renamed from D9; footprint SparkFun-LED:LED_0603_1608Metric_Red -> LED_SMD:LED_0201_0603Metric_Pad0.64x0.40mm_HandSolder; symbol SparkFun-LED:LED_Red_0603 -> PCM_SparkFun-LED:LED_Red_0603
- D5: renamed from D7; footprint SparkFun-LED:LED_0603_1608Metric_Red -> LED_SMD:LED_0201_0603Metric_Pad0.64x0.40mm_HandSolder; symbol SparkFun-LED:LED_Red_0603 -> PCM_SparkFun-LED:LED_Red_0603
- D6: renamed from D5; footprint PCM_Diode_SMD_AKL:D_SOD-523 -> Diode_SMD:D_SOD-523
- D7: renamed from D8; footprint SparkFun-LED:LED_0603_1608Metric_Red -> LED_SMD:LED_0201_0603Metric_Pad0.64x0.40mm_HandSolder; symbol SparkFun-LED:LED_Red_0603 -> PCM_SparkFun-LED:LED_Red_0603
- D8: renamed from D6; footprint PCM_Diode_SMD_AKL:D_SOD-523 -> Diode_SMD:D_SOD-523
- DV1, DV2, DV3: footprint ItlaModules:PHE-3A -> ITLA_Modules:PHE-3A; symbol Itla_Modules:PHE-3A -> ITLA_Modules:PHE-3A
- R1: footprint Resistor_SMD_AKL:R_0603_1608Metric -> EasyEDA:R0603
- R10: renamed from R16; footprint Resistor_SMD_AKL:R_0603_1608Metric -> EasyEDA:R0603
- R11: renamed from R13; footprint PCM_Resistor_SMD_AKL:R_0603_1608Metric -> EasyEDA:R0603
- R12: renamed from R14; footprint PCM_Resistor_SMD_AKL:R_0603_1608Metric -> EasyEDA:R0603
- R13: renamed from R9; footprint PCM_Resistor_SMD_AKL:R_0603_1608Metric -> EasyEDA:R0603
- R14: renamed from R10; footprint PCM_Resistor_SMD_AKL:R_0603_1608Metric -> EasyEDA:R0603
- R15: renamed from R11; footprint PCM_Resistor_SMD_AKL:R_0603_1608Metric -> EasyEDA:R0603
- R16: renamed from R12; footprint PCM_Resistor_SMD_AKL:R_0603_1608Metric -> EasyEDA:R0603
- R17: renamed from R7; footprint PCM_Resistor_SMD_AKL:R_0603_1608Metric -> EasyEDA:R0603
- R18: renamed from R8; footprint PCM_Resistor_SMD_AKL:R_0603_1608Metric -> EasyEDA:R0603
- R2: footprint PCM_Resistor_SMD_AKL:R_0603_1608Metric -> EasyEDA:R0603
- R4: renamed from R3; footprint PCM_Resistor_SMD_AKL:R_0603_1608Metric -> EasyEDA:R0603
- R5: renamed from R17; footprint Resistor_SMD_AKL:R_0603_1608Metric -> EasyEDA:R0603
- R6: renamed from R4; footprint PCM_Resistor_SMD_AKL:R_0603_1608Metric -> EasyEDA:R0603
- R7: renamed from R5; footprint PCM_Resistor_SMD_AKL:R_0603_1608Metric -> EasyEDA:R0603
- R8: renamed from R15; footprint Resistor_SMD_AKL:R_0603_1608Metric -> EasyEDA:R0603
- R9: renamed from R6; footprint PCM_Resistor_SMD_AKL:R_0603_1608Metric -> EasyEDA:R0603
- renumbered J5 to J6
Connections:
- net +24V: now also D2.2, Q2.3 (S), R3.1; no longer DV1.12 (VCC), DV1.8 (VCC), DV2.12 (VCC), DV2.8 (VCC), DV3.12 (VCC), DV3.8 (VCC)
- net +3.3V: now also J5.1 (Pin_1); no longer DV1.4 (Vref), DV2.4 (Vref), DV3.4 (Vref)
- net ACT_1: now also Q3.1
- net ACT_2: now also Q4.1
- net ACT_3: now also Q5.1
- net BOOT: now also R1.2, C2.1, SW1.1; no longer R2.2
- net GND: now also C2.2, C3.1, Q3.2, Q4.2, Q5.2, SW1.2, SW2.2, USB1.1 (GND), USB1.12 (GND), USB1.13 (SHELL), USB1.14 (SHELL)
- net MOTOR1_A: now also J3.1 (Pin_1)
- net MOTOR1_B: now also J3.2 (Pin_2)
- net MOTOR2_A: now also J2.1 (Pin_1)
- net MOTOR2_B: now also J2.2 (Pin_2)
- net MOTOR3_A: now also J4.1 (Pin_1)
- net MOTOR3_B: now also J4.2 (Pin_2)
- net VBUS: now also D3.1, USB1.11 (VBUS), USB1.2 (VBUS)
- net VCC: now also D2.1, D3.2
- net at R4.1: now also USB1.4 (CC1)
- net at R9.1: now also USB1.6 (DP1), USB1.8 (DP2)
- net at R7.1: now also USB1.5 (DN2), USB1.7 (DN1)
- net at R6.1: now also USB1.10 (CC2)
- net EN renamed CHIP_PU
- net CHIP_PU: now also R2.2, C3.2, SW2.1; no longer R1.2
- new net: DV2.4 (Vref), TP2.1
- new net: DV3.4 (Vref), TP3.1
- new net: DV1.4 (Vref), TP1.1
- new net: J5.2 (Pin_2), Q3.3
- new net: J5.3 (Pin_3), Q4.3
- new net: Q2.1 (G), Q5.3, R3.2
- new net V_DRIVER: DV1.12 (VCC), DV1.8 (VCC), DV2.12 (VCC), DV2.8 (VCC), DV3.12 (VCC), DV3.8 (VCC), Q2.2 (D)
Other:
- note added: "3.3V Switches"
- note added: "ALIMENTACION"
- note added: "Active High 50V 100mA"
- note added: "BTN RST & BOOT"
- note added: "CONEXIONES SENSORES"
- note added: "DC-DC STEP-DOWN"
- note added: "DRIVERS"
- note added: "ENCENDIDO SECUENCIAL"
- note added: "INDICADORES DE VOLTAJES"
- note added: "MCU"
- note added: "Mecanico"
- note added: "PROTECCION TVS MCU"
- note added: "PULL-UP UART SENSOR-CO^{2}"
- note added: "USB-C"
- note removed: "OUTPUT DIGITALES OPEN COLECTOR STM-COMMUNICATION"
- note removed: "UART SENSOR-CO^{2}"
- moved on the sheet: C10, C11, C12, C13, C14, C15, C16, C4, C5, C6, C7, C8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
